Commit message: tried some stuff

File: spot_v1_description/urdf/spot_v1.urdf (robot description, URDF)
Before this commit: robot spot_v1, 15 links, 14 joints
Links:
- link base_imu: geometry collision mesh filename=meshes/base_imu_1.stl scale=0.001 0.001 0.001; visual mesh filename=meshes/base_imu_1.stl scale=0.001 0.001 0.001
- link base_laser_1: geometry collision mesh filename=meshes/base_laser_1.stl scale=0.001 0.001 0.001; visual mesh filename=meshes/base_laser_1.stl scale=0.001 0.001 0.001
- link base_link: geometry collision mesh filename=meshes/base_link.stl scale=0.001 0.001 0.001; visual mesh filename=meshes/base_link.stl scale=0.001 0.001 0.001
- link elbow_bl_5: geometry collision mesh filename=meshes/elbow_bl_5.stl scale=0.001 0.001 0.001; visual mesh filename=meshes/elbow_bl_5.stl scale=0.001 0.001 0.001
- link elbow_br_1: geometry collision mesh filename=meshes/elbow_br_1.stl scale=0.001 0.001 0.001; visual mesh filename=meshes/elbow_br_1.stl scale=0.001 0.001 0.001
- link elbow_fl_1: geometry collision mesh filename=meshes/elbow_fl_1.stl scale=0.001 0.001 0.001; visual mesh filename=meshes/elbow_fl_1.stl scale=0.001 0.001 0.001
- link elbow_fr_1: geometry collision mesh filename=meshes/elbow_fr_1.stl scale=0.001 0.001 0.001; visual mesh filename=meshes/elbow_fr_1.stl scale=0.001 0.001 0.001
- link lower_bl_1: geometry collision mesh filename=meshes/lower_bl_1.stl scale=0.001 0.001 0.001; visual mesh filename=meshes/lower_bl_1.stl scale=0.001 0.001 0.001
- link lower_br_1: geometry collision mesh filename=meshes/lower_br_1.stl scale=0.001 0.001 0.001; visual mesh filename=meshes/lower_br_1.stl scale=0.001 0.001 0.001
- link lower_fl_1: geometry collision mesh filename=meshes/lower_fl_1.stl scale=0.001 0.001 0.001; visual mesh filename=meshes/lower_fl_1.stl scale=0.001 0.001 0.001
- link lower_fr_1: geometry collision mesh filename=meshes/lower_fr_1.stl scale=0.001 0.001 0.001; visual mesh filename=meshes/lower_fr_1.stl scale=0.001 0.001 0.001
- link upper_bl_1: geometry collision mesh filename=meshes/upper_bl_1.stl scale=0.001 0.001 0.001; visual mesh filename=meshes/upper_bl_1.stl scale=0.001 0.001 0.001
- link upper_br_1: geometry collision mesh filename=meshes/upper_br_1.stl scale=0.001 0.001 0.001; visual mesh filename=meshes/upper_br_1.stl scale=0.001 0.001 0.001
- link upper_fl_1: geometry collision mesh filename=meshes/upper_fl_1.stl scale=0.001 0.001 0.001; visual mesh filename=meshes/upper_fl_1.stl scale=0.001 0.001 0.001
- link upper_fr_1: geometry collision mesh filename=meshes/upper_fr_1.stl scale=0.001 0.001 0.001; visual mesh filename=meshes/upper_fr_1.stl scale=0.001 0.001 0.001
