Commit message: fixed command, observation, reward and class config

File: ressources/urdfs/spot/spot_v2.urdf (robot description, URDF)
Before this commit: robot spot_v1, 15 links, 14 joints
Links:
- removed link base_imu
- removed link base_laser_1
Joints:
- removed joint Rigid 48
- removed joint Rigid 49

Commit message: fixing some bugs

File: ressources/urdfs/spot/spot_v2.urdf (robot description, URDF)
Before this commit: robot spot_v1, 13 links, 12 joints
Joints:
- joint Revolute 30: origin xyz=-0.038998 -0.0085 0.0 rpy=0 0 0 -> xyz=-0.038998 -0.0085 0.0 rpy=0.8 0 0
- joint Revolute 32: origin xyz=-0.038998 0.0085 0.0 rpy=0 0 0 -> xyz=-0.038998 0.0085 0.0 rpy=0.8 0 0
- joint Revolute 35: origin xyz=0.038998 -0.0085 0.0 rpy=0 0 0 -> xyz=0.038998 -0.0085 0.0 rpy=0.8 0 0
- joint Revolute 36: origin xyz=0.038998 0.0085 0.0 rpy=0 0 0 -> xyz=0.038998 0.0085 0.0 rpy=0.8 0 0

Commit message: fix urdf

File: ressources/urdfs/spot/spot_v2.urdf (robot description, URDF)
Before this commit: robot spot_v1, 13 links, 12 joints
Links:
- link base_link: mass 4.569295440014468 -> 3.569295440014468
Joints:
- joint Revolute 29: limit lower=-0.872665 upper=0.785398 effort=1.47 velocity=6.5 -> lower=-0.872665 upper=0.5085398 effort=1.47 velocity=4.5; origin xyz=-0.003 0.024449 -0.083518 rpy=0 0 0 -> xyz=-0.003 0.024449 -0.083518 rpy=-0.2 0 0
- joint Revolute 30: limit lower=0.523599 upper=3.316126 effort=1.72 velocity=6.5 -> lower=0.223599 upper=1.516126 effort=1.72 velocity=4.5; origin xyz=-0.038998 -0.0085 0.0 rpy=0.8 0 0 -> xyz=-0.038998 -0.0085 0.0 rpy=-0.5 0 0
- joint Revolute 32: limit lower=0.523599 upper=3.316126 effort=1.72 velocity=6.5 -> lower=0.223599 upper=1.516126 effort=1.72 velocity=4.5; origin xyz=-0.038998 0.0085 0.0 rpy=0.8 0 0 -> xyz=-0.038998 0.0085 0.0 rpy=-0.5 0 0
- joint Revolute 33: limit lower=-0.872665 upper=0.785398 effort=1.72 velocity=6.5 -> lower=-0.872665 upper=0.5085398 effort=1.72 velocity=4.5; origin xyz=-0.003 0.02445 -0.083518 rpy=0 0 0 -> xyz=-0.003 0.02445 -0.083518 rpy=-0.2 0 0
- joint Revolute 35: limit lower=-3.316126 upper=-0.523599 effort=1.72 velocity=6.5 -> lower=-1.516126 upper=-0.223599 effort=1.72 velocity=4.5; origin xyz=0.038998 -0.0085 0.0 rpy=0.8 0 0 -> xyz=0.038998 -0.0085 0.0 rpy=-0.5 0 0
- joint Revolute 36: limit lower=-3.316126 upper=-0.523599 effort=1.72 velocity=6.5 -> lower=-1.516126 upper=-0.223599 effort=1.72 velocity=4.5; origin xyz=0.038998 0.0085 0.0 rpy=0.8 0 0 -> xyz=0.038998 0.0085 0.0 rpy=-0.5 0 0
- joint Revolute 37: limit lower=-0.872665 upper=0.785398 effort=1.47 velocity=6.5 -> lower=-0.872665 upper=0.5085398 effort=1.47 velocity=4.5; origin xyz=0.003 0.024449 -0.083518 rpy=0 0 0 -> xyz=0.003 0.024449 -0.083518 rpy=-0.2 0 0
- joint Revolute 38: limit lower=-0.872665 upper=0.785398 effort=1.72 velocity=6.5 -> lower=-0.872665 upper=0.5085398 effort=1.72 velocity=4.5; origin xyz=0.003 0.02445 -0.083518 rpy=0 0 0 -> xyz=0.003 0.02445 -0.083518 rpy=-0.2 0 0
- joint Revolute 43: limit lower=-1.570796 upper=1.570796 effort=1.37 velocity=6.5 -> lower=-0.370796 upper=0.370796 effort=1.37 velocity=4.5
- joint Revolute 45: limit lower=-1.570796 upper=1.570796 effort=1.37 velocity=6.5 -> lower=-0.370796 upper=0.370796 effort=1.37 velocity=4.5
- joint Revolute 46: limit lower=-1.570796 upper=1.570796 effort=1.37 velocity=6.5 -> lower=-0.370796 upper=0.370796 effort=1.37 velocity=4.5
- joint Revolute 47: limit lower=-1.570796 upper=1.570796 effort=1.37 velocity=6.5 -> lower=-0.570796 upper=0.370796 effort=1.37 velocity=4.5
